File: hardware/psp-bluetooth/psp-bluetooth.kicad_sch (KiCad schematic)
At the start: 2 parts, among them J1 Conn_01x10_Female

Commit message: Added Mappings (#2)
* Initial work and hardware stuff

* Move around stuff

* Adding mappings for analogue sticks

* Added PCB pinout

* Final
Parts:
- removed A1: Arduino_Nano_v3.x, Module:Arduino_Nano, symbol MCU_Module:Arduino_Nano_v3.x
- removed J1: Conn_01x10_Female, symbol Connector:Conn_01x10_Female
- added J1: Left Connector, Connector_FFC-FPC:Hirose_FH12-10S-0.5SH_1x10-1MP_P0.50mm_Horizontal, symbol Connector_Generic:Conn_01x10
- added J2: Center Connector, Connector_FFC-FPC:Hirose_FH12-10S-0.5SH_1x10-1MP_P0.50mm_Horizontal, symbol Connector_Generic:Conn_01x10
- added J3: Right Connector, Connector_FFC-FPC:Hirose_FH12-14S-0.5SH_1x14-1MP_P0.50mm_Horizontal, symbol Connector_Generic:Conn_01x14
- added J4: Analog Connector, Connector_PinHeader_2.54mm:PinHeader_1x04_P2.54mm_Vertical, symbol Connector_Generic:Conn_01x04
- added J5: PSP Power out, Connector_PinHeader_2.54mm:PinHeader_1x02_P2.54mm_Vertical, symbol Connector_Generic:Conn_01x02
- added J6: Barrel_Jack, Connector_BarrelJack:BarrelJack_CUI_PJ-063AH_Horizontal, symbol Connector:Barrel_Jack
- added J7: Serial, Connector_PinHeader_2.54mm:PinHeader_1x02_P2.54mm_Vertical, symbol Connector_Generic:Conn_01x02
- added J8: Vin Toggle, Connector_PinHeader_2.54mm:PinHeader_1x02_P2.54mm_Vertical, symbol Connector_Generic:Conn_01x02
- added JP1: SJ Vin Toggle, Jumper:SolderJumper-2_P1.3mm_Open_Pad1.0x1.5mm, symbol Jumper:SolderJumper_2_Open
- added P1: Digital, Socket_Arduino_Nano:Socket_Strip_Arduino_1x15, symbol Connector_Generic:Conn_01x15
- added P2: Analog, Socket_Arduino_Nano:Socket_Strip_Arduino_1x15, symbol Connector_Generic:Conn_01x15
- added P3, P4, P5, P6: CONN_01X01, Socket_Arduino_Nano:1pin_Nano, symbol Connector_Generic:Conn_01x01
- added S1: L102021ML04Q, L102021ML04Q:SW_L102021ML04Q, symbol L102021ML04Q:L102021ML04Q
- added SW1: SW_Push, Button_Switch_SMD:SW_Push_1P1T_NO_6x6mm_H9.5mm, symbol Switch:SW_Push
- added U1: MCP4251-xxxx-P, Package_DIP:DIP-14_W7.62mm, symbol Potentiometer_Digital:MCP4251-xxxx-P
Connections:
- new net: J5.2 (Pin_2), J8.1 (Pin_1), JP1.1 (A), S1.2
- new net: J6.2, S1.3
- new net +3V3: P2.14 (Pin_14), U1.14 (VDD)
- new net +5V: P2.4 (Pin_4)
- new net 0(Rx): J7.2 (Pin_2), P1.2 (Pin_2)
- new net 1(Tx): J7.1 (Pin_1), P1.1 (Pin_1)
- new net 10(**/SS): P1.13 (Pin_13)
- new net 10(**/SS): U1.1 (~{CS})
- new net 11(**/MOSI): P1.14 (Pin_14)
- new net 11(**/MOSI): U1.3 (SDI)
- new net 12(MISO): P1.15 (Pin_15), U1.13 (SDO)
- new net 13(SCK): P2.15 (Pin_15), U1.2 (SCK)
- new net 2: J3.5 (Pin_5), P1.5 (Pin_5)
- new net 3(**): J3.4 (Pin_4), P1.6 (Pin_6)
- new net 4: J3.3 (Pin_3), P1.7 (Pin_7)
- new net 5(**): J3.2 (Pin_2), P1.8 (Pin_8)
- new net 6(**): J1.10 (Pin_10), P1.9 (Pin_9)
- new net 7: J1.8 (Pin_8), P1.10 (Pin_10)
- new net 8: J1.7 (Pin_7), P1.11 (Pin_11)
- new net 9(**): J1.6 (Pin_6), P1.12 (Pin_12)
- new net A0 (D14): J2.10 (Pin_10), P2.12 (Pin_12)
- new net A1 (D15): J2.9 (Pin_9), P2.11 (Pin_11)
- new net A2 (D16): J2.7 (Pin_7), P2.10 (Pin_10)
- new net A3 (D17): J2.1 (Pin_1), P2.9 (Pin_9)
- new net A4 (D18): J1.9 (Pin_9), P2.8 (Pin_8)
- new net A5 (D19): J3.1 (Pin_1), P2.7 (Pin_7)
- new net A6 (D20): P2.6 (Pin_6), SW1.1
- new net A7 (D21): J3.10 (Pin_10), P2.5 (Pin_5)
- new net AREF: P2.13 (Pin_13)
- new net GND: J1.1 (Pin_1), J1.2 (Pin_2), J1.3 (Pin_3), J1.4 (Pin_4), J1.5 (Pin_5), J2.4 (Pin_4), J2.5 (Pin_5), J2.6 (Pin_6), J3.6 (Pin_6), J3.7 (Pin_7), J3.8 (Pin_8), J3.9 (Pin_9), J4.1 (Pin_1), J5.1 (Pin_1), J6.1, P1.4 (Pin_4), P2.2 (Pin_2), SW1.2, U1.10 (P0B), U1.4 (VSS), U1.5 (P1B)
- new net P0A/P1A: J4.3 (Pin_3), U1.7 (P1A), U1.8 (P0A)
- new net P0W: J4.4 (Pin_4), U1.9 (P0W)
- new net P1W: J4.2 (Pin_2), U1.6 (P1W)
- new net Reset: P1.3 (Pin_3), P2.3 (Pin_3)
- new net VIN: J8.2 (Pin_2), JP1.2 (B), P2.1 (Pin_1)
- no-connect marks 0 -> 17
Other:
- note added: "1"
- note added: "Arduino Nano"
- note added: "Holes"
