File: hardware - v3/psp-bluetooth/psp-bluetooth.kicad_pcb (KiCad board)
At the start: 2 copper layers, 91.4 x 71.1 mm, 22 parts, among them J1 Left Connector, J2 Center Connector, J3 Right Connector, J4 Analog Connector, J5 PSP Power out, J6 Barrel_Jack, J8 Vin Toggle, P1 Digital, P2 Analog, SW1 SW_Push, U1 MCP4251-xxxx-P

Commit message: Finished
Parts:
- removed S2: L102021ML04Q, L102021ML04Q:SW_L102021ML04Q
- added G***: LOGO, Graphics:pcblogo, F.Cu at (138.0, 83.0)
- added J7: Programming Header 1, Connector_PinHeader_2.54mm:PinHeader_1x02_P2.54mm_Vertical, F.Cu at (176.5, 45.7)
- JP2: value SJ Vin Toggle -> SJ LED Indicator
- moved JP2 6.80 mm to (176.5, 40.5)
- moved SW1 4.12 mm to (189.5, 34.5)
Routing:
- net /A6 (D20): track 72.5 -> 60.7 mm
- net /1(Tx): track 46.1 -> 34.9 mm
- net Net-(J7-Pad1): track 20.5 -> 15.1 mm
Other:
- board text added: "Following FFC & Connector types [MUST] be used * Type A FFC & Top Interfacing Connector * Type D FFC & Bottom Interfacing Connector"
- board text added: "IMPORTANT"
- board text added: "PROG TGL 1"
- board text added: "PROG TGL 1 [MUST] be disconnected when programming"
- board text added: "PWR TGL 1"
- board text added: "PWR TGL 1 [MUST] be disconnected when powered via USB"
- board text added: "https://github.com/ste2425/PSP-Bluetooth-Controller"
- board text removed: "Normal Mode"
- board text removed: "Programming Mode"
