File: hardware/buttonsSuper/buttonsSuper.kicad_sch (KiCad schematic)
At the start: 19 parts, among them P1 5034801000

Commit message: wip
Parts:
- removed C7: flex-conector_10, consolizer:flex_long_10, symbol consolizer:flex-conector_10
- removed CIRCLE1, CROSS1, DOWN1, L1, LEFT1, R1, RIGHT1, SQUARE1, TRIANGLE1, UP1: K2-1187SQ-E4SW-06, JLCPCB_footprint:KEY-SMD_4P-L5.2-W5.2-P3.70-LS6.4_1, symbol JLCPCB_schematic:K2-1187SQ-E4SW-06
- removed P1: 5034801000, JLCPCB_footprint:FPC-SMD_5034801000, symbol JLCPCB_schematic:5034801000
- added C10: flex-conector_10, consolizer:flex_long_10, symbol consolizer:PSP-Analog-FFC-Male
- added C9: flex-conector_10, consolizer:flex_short_10, symbol consolizer:flex-conector_10
- added DOWN1, L1, L2, L3, L4, L5, L6, LEFT1, RIGHT1, UP1: SKRRABE010, JLCPCB_footprint:KEY-SMD_4P-L5.2-W5.2-P3.70-LS6.4_1, symbol JLCPCB_schematic2:SKRRABE010_2pin
- added U1, U2, U3, U4, U5, U6, U7: SKRBAAE010, JLCPCB_footprint:KEY-SMD_4P-L4.8-W4.8-P3.65_SKRBAAE010, symbol JLCPCB_schematic2:SKRBAAE010
Connections:
- net +v: now also C10.2 (+v)
- net Circle: now also L6.1
- net GND: now also DOWN1.2, L1.2, LEFT1.2, RIGHT1.2, UP1.2; no longer C6.1 (GND_[1]), C6.5 (GND_[2])
- net R1: now also L3.1
- net Square: now also L5.1
- net Triangle: now also L4.1
- net cross: now also L2.1
- net down: now also DOWN1.1
- net gnd: now also L2.2, L3.2, L4.2, L5.2, L6.2
- net l1: now also L1.1
- net left: now also LEFT1.1
- net right: now also RIGHT1.1
- net up: now also UP1.1
- net start: now reaches C8.1
- net start: now also C9.1, U3.2, U3.4
- net home: now reaches C8.10
- net home: now also C9.10, U7.2, U7.4
- net select: now reaches C8.2
- net select: now also C9.2, U4.2, U4.4
- net music: now reaches C8.3
- net music: now also C9.3, U1.2, U1.4
- net gnd2: now reaches C8.4
- net gnd2: now also C8.5, C8.6, C9.4, C9.5, C9.6, U1.1, U1.3, U2.1, U2.3, U3.1, U3.3, U4.1, U4.3, U5.1, U5.3, U6.1, U6.3, U7.1, U7.3
- net screen: now reaches C8.7
- net screen: now also C9.7, U2.2, U2.4
- net vol up: now reaches C8.8
- net vol up: now also C9.8, U5.2, U5.4
- net vol down: now reaches C8.9
- net vol down: now also C9.9, U6.2, U6.4
- net X_1 renamed analog_x
- net analog_x: now also C10.3 (Analog_X)
- net X_2 renamed PSP_x
- net PSP_x: now also C10.9 (PSP_x)
- net Y_1 renamed Analog_y
- net Analog_y: now also C10.1 (Analog_y)
- net Y_2 renamed PSP_y
- net PSP_y: now also C10.10 (PSP_y)
- new net gnd3: C10.4 (gnd), C6.1 (Analog_gnd), C6.5 (PSP_gnd)
- no-connect marks 5 -> 1
Other:
- moved on the sheet: C1, C2, C6
