File: hardware/esp/esp32/changes.kicad_sch (KiCad schematic)
At the start: 0 parts

Commit message: stuff
Other:
- note removed: "V0.2: Modified power caps. Repalced 1500uf for 22uf and 10 uf. Removed current limiting resistors for PSPpower and PSP screen on detect, Added diodes instead."
Changed lines of the file:
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@@
 		(comment 4 "UNDER REVIEW - SUBJECT TO CHANGE")
 	)
-	(text "V0.2:\nModified power caps. Repalced 1500uf for 22uf and 10 uf.\n\nRemoved current limiting resistors for PSPpower and PSP screen on detect,\nAdded diodes instead."
-		(exclude_from_sim no)
-		(at 52.578 23.114 0)
-		(effects
-			(font
-				(size 1.27 1.27)
-			)
-		)
-	)
 )
